Commit message: Bump version 0.2.6 fixes: URDF naming, mapping launch, simulator precision

File: urdf/tango.urdf (robot description, URDF)
Before this commit: robot tango_robot, 7 links, 6 joints
Links:
- removed link lidar_link
- added link laser_link, mass 0.2; collision cylinder length=0.050 radius=0.040; visual box size=0.090 0.090 0.010
Joints:
- removed joint lidar_joint
- added joint laser_joint: type fixed, parent base_link, child laser_link, origin xyz=-0.025 0.000 0.165 rpy=0 0 0
- joint wheel_front_left_joint: origin xyz=0.100 0.1625 0.040 rpy=0 0 0 -> xyz=0.000 0.1625 0.040 rpy=0 0 0
- joint wheel_front_right_joint: origin xyz=0.100 -0.1625 0.040 rpy=0 0 0 -> xyz=0.000 -0.1625 0.040 rpy=0 0 0
- joint wheel_rear_left_joint: origin xyz=-0.100 0.1625 0.040 rpy=0 0 0 -> xyz=-0.200 0.1625 0.040 rpy=0 0 0
- joint wheel_rear_right_joint: origin xyz=-0.100 -0.1625 0.040 rpy=0 0 0 -> xyz=-0.200 -0.1625 0.040 rpy=0 0 0
